File: hardware/_rotary_.kicad_pcb (KiCad board)
At the start: 2 copper layers, 40 x 80 mm, 32 parts, among them J1 mono_jack_3.5mm, J2 jst_xa_3, SW1 SW_DPDT_x2, U1 TLV2372, U2 LM317, U3 TLV2374

Commit message: update pcbs and panels
Parts:
- R13: value 2.5k -> 2.4k
- RV1: value 1k_pot -> 1k_pot_d
- RV3: value 100k -> 100k_pot
- moved R14 0.57 mm to (83.7, 114.1)
Other:
- outline, holes or cut-outs redrawn
- board text added: "_rotary_ v1_1_1 cyberboy666 & autr"
- board text removed: "_rotary_ v1_1_0 cyberboy666 & autr"
